File: sens-rf-1w-1-kicad/sens-rf-1w-1-kicad.kicad_pcb (KiCad board)
At the start: 2 copper layers, 251.4 x 39.4 mm, 67 parts, among them J1 I2C, J2 I2C, J3 I2C, J4 Debug port, J5 SPI / GPIO, J7 U.FL, SW1 Next, SW2 Select, SW3 Reset, U1 AMS1117-3.3

Commit message: First cut at the Makefile
Other:
- board text added: "300 mA"
